File: PCB/Eagle/Arduino_AMRSID_tester_dual.brd (EAGLE design)
At the start: 59.7 x 53.3 mm, 21 parts

Commit message: Schematic update for better readability
Connections:
- net N$3 renamed AUD-R
- net N$5 renamed POTX-1
- net N$6 renamed POTY-1
- net N$7 renamed AUD-L
- net N$8 renamed POTX-2
- net N$9 renamed POTY-2
Changed lines of the file:
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@@
 <?xml version="1.0" encoding="utf-8"?>
 <!DOCTYPE eagle SYSTEM "eagle.dtd">
-<eagle version="9.5.2">
+<eagle version="6.5.0">
 <drawing>
 <settings>
 <setting alwaysvectorfont="no"/>
-<setting keepoldvectorfont="yes"/>
 <setting verticaltext="up"/>
 </settings>
@@
 <param name="dpMaxLengthDifference" value="10mm"/>
 <param name="dpGapFactor" value="2.5"/>
+<param name="checkGrid" value="0"/>
 <param name="checkAngle" value="0"/>
 <param name="checkFont" value="1"/>
 <param name="checkRestrict" value="0"/>
-<param name="checkStop" value="0"/>
-<param name="checkValues" value="0"/>
-<param name="checkNames" value="1"/>
-<param name="checkWireStubs" value="1"/>
-<param name="checkPolygonWidth" value="0"/>
 <param name="useDiameter" value="13"/>
 <param name="maxErrors" value="50"/>
@@
 <pass name="Default">
 <param name="RoutingGrid" value="50mil"/>
-<param name="AutoGrid" value="1"/>
-<param name="Efforts" value="0"/>
-<param name="TopRouterVariant" value="1"/>
 <param name="tpViaShape" value="round"/>
-<param name="PrefDir.1" value="a"/>
+<param name="PrefDir.1" value="|"/>
 <param name="PrefDir.2" value="0"/>
 <param name="PrefDir.3" value="0"/>
@@
 <param name="PrefDir.14" value="0"/>
 <param name="PrefDir.15" value="0"/>
-<param name="PrefDir.16" value="a"/>
+<param name="PrefDir.16" value="-"/>
 <param name="cfVia" value="8"/>
 <param name="cfNonPref" value="5"/>
@@
 <wire x1="36.83" y1="27.305" x2="36.83" y2="30.48" width="0.3048" layer="1"/>
 </signal>
-<signal name="N$3">
+<signal name="AUD-R">
 <contactref element="SOCKET" pad="6"/>
 <contactref element="C8" pad="+"/>
@@
 <wire x1="1.836" y1="20.251" x2="1.836" y2="12.369" width="0.6096" layer="1"/>
 </signal>
-<signal name="N$8">
+<signal name="POTX-2">
 <contactref element="R3" pad="1"/>
 <contactref element="C5" pad="2"/>
@@
 <wire x1="39.37" y1="38.735" x2="39.37" y2="39.64" width="0.3048" layer="16"/>
 </signal>
-<signal name="N$9">
+<signal name="POTY-2">
 <contactref element="C6" pad="2"/>
 <contactref element="R4" pad="1"/>
@@
 <wire x1="35.56" y1="38.735" x2="35.56" y2="39.64" width="0.3048" layer="16"/>
 </signal>
-<signal name="N$5">
+<signal name="POTX-1">
 <contactref element="R1" pad="1"/>
 <contactref element="C3" pad="2"/>
@@
 <wire x1="39.37" y1="15.875" x2="39.37" y2="16.78" width="0.3048" layer="16"/>
 </signal>
-<signal name="N$6">
+<signal name="POTY-1">
 <contactref element="R2" pad="1"/>
 <contactref element="C4" pad="2"/>
@@
 <wire x1="6.985" y1="45.72" x2="8.89" y2="43.815" width="0.6096" layer="16"/>
 </signal>
-<signal name="N$7">
+<signal name="AUD-L">
 <contactref element="C7" pad="+"/>
 <contactref element="ARM2SID" pad="27"/>
@@
 </signal>
 </signals>
-<mfgpreviewcolors>
-<mfgpreviewcolor name="soldermaskcolor" color="0xC8008000"/>
-<mfgpreviewcolor name="silkscreencolor" color="0xFFFEFEFE"/>
-<mfgpreviewcolor name="backgroundcolor" color="0xFF282828"/>
-<mfgpreviewcolor name="coppercolor" color="0xFFFFBF00"/>
-<mfgpreviewcolor name="substratecolor" color="0xFF786E46"/>
-</mfgpreviewcolors>
 </board>
 </drawing>

Commit message: SCH and PCB update
Parts:
- C10, C11, C12, C9: value 15n -> n.c.
- moved AUDIO1 0.30 mm to (5.00, 52.7)
Connections:
- net POTX-1 renamed POTX-L
- net POTX-2 renamed POTX-R
- net POTY-1 renamed POTY-L
- net POTY-2 renamed POTY-R
Other:
- outline, holes or cut-outs redrawn
Changed lines of the file:
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@@
 <?xml version="1.0" encoding="utf-8"?>
 <!DOCTYPE eagle SYSTEM "eagle.dtd">
-<eagle version="6.5.0">
+<eagle version="9.5.2">
 <drawing>
 <settings>
 <setting alwaysvectorfont="no"/>
+<setting keepoldvectorfont="yes"/>
 <setting verticaltext="up"/>
 </settings>
-<grid distance="50" unitdist="mil" unit="mil" style="dots" multiple="5" display="yes" altdistance="0.025" altunitdist="inch" altunit="mm"/>
+<grid distance="32" unitdist="mil" unit="mil" style="dots" multiple="5" display="yes" altdistance="0.025" altunitdist="inch" altunit="mm"/>
 <layers>
 <layer number="1" name="Top" color="4" fill="1" visible="yes" active="yes"/>
@@
 <layer number="21" name="tPlace" color="7" fill="1" visible="yes" active="yes"/>
 <layer number="22" name="bPlace" color="7" fill="1" visible="yes" active="yes"/>
-<layer number="23" name="tOrigins" color="15" fill="1" visible="no" active="yes"/>
+<layer number="23" name="tOrigins" color="15" fill="1" visible="yes" active="yes"/>
 <layer number="24" name="bOrigins" color="15" fill="1" visible="no" active="yes"/>
 <layer number="25" name="tNames" color="7" fill="1" visible="yes" active="yes"/>
@@
 <wire x1="57.15" y1="0" x2="2.54" y2="0" width="0.0762" layer="20"/>
 <wire x1="2.54" y1="0" x2="0" y2="2.54" width="0.0762" layer="20"/>
-<wire x1="0" y1="2.54" x2="0" y2="50.8" width="0.0762" layer="20"/>
+<wire x1="0" y1="2.54" x2="0" y2="29.2608" width="0.0762" layer="20"/>
+<wire x1="0" y1="29.2608" x2="0.8128" y2="30.0736" width="0.0762" layer="20"/>
+<wire x1="0.8128" y1="30.0736" x2="0.8128" y2="45.5168" width="0.0762" layer="20"/>
+<wire x1="0.8128" y1="45.5168" x2="0" y2="46.3296" width="0.0762" layer="20"/>
+<wire x1="0" y1="46.3296" x2="0" y2="50.8" width="0.0762" layer="20"/>
 <wire x1="0" y1="50.8" x2="2.54" y2="53.34" width="0.0762" layer="20"/>
 <rectangle x1="15.097125" y1="0.714375" x2="15.160625" y2="0.746125" layer="25"/>
@@
 <param name="dpMaxLengthDifference" value="10mm"/>
 <param name="dpGapFactor" value="2.5"/>
-<param name="checkGrid" value="0"/>
 <param name="checkAngle" value="0"/>
 <param name="checkFont" value="1"/>
 <param name="checkRestrict" value="0"/>
+<param name="checkStop" value="0"/>
+<param name="checkValues" value="0"/>
+<param name="checkNames" value="1"/>
+<param name="checkWireStubs" value="1"/>
+<param name="checkPolygonWidth" value="0"/>
 <param name="useDiameter" value="13"/>
 <param name="maxErrors" value="50"/>
@@
 <pass name="Default">
 <param name="RoutingGrid" value="50mil"/>
+<param name="AutoGrid" value="1"/>
+<param name="Efforts" value="0"/>
+<param name="TopRouterVariant" value="1"/>
 <param name="tpViaShape" value="round"/>
-<param name="PrefDir.1" value="|"/>
+<param name="PrefDir.1" value="a"/>
 <param name="PrefDir.2" value="0"/>
 <param name="PrefDir.3" value="0"/>
@@
 <param name="PrefDir.14" value="0"/>
 <param name="PrefDir.15" value="0"/>
-<param name="PrefDir.16" value="-"/>
+<param name="PrefDir.16" value="a"/>
 <param name="cfVia" value="8"/>
 <param name="cfNonPref" value="5"/>
@@
 <attribute name="VALUE" x="10.75" y="49.915" size="1.27" layer="28" rot="MR180"/>
 </element>
-<element name="C9" library="rcl" package="C0805K" value="15n" x="20.32" y="10.795" smashed="yes" rot="MR0">
+<element name="C9" library="rcl" package="C0805K" value="n.c." x="20.32" y="10.795" smashed="yes" rot="MR0">
 <attribute name="NAME" x="21.32" y="11.924" size="1.27" layer="26" font="vector" ratio="15" rot="MR0"/>
 <attribute name="VALUE" x="21.32" y="8.895" size="1.016" layer="28" rot="MR0"/>
 </element>
-<element name="C10" library="rcl" package="C0805K" value="15n" x="25.4" y="10.795" smashed="yes" rot="MR0">
+<element name="C10" library="rcl" package="C0805K" value="n.c." x="25.4" y="10.795" smashed="yes" rot="MR0">
 <attribute name="NAME" x="26.908" y="11.797" size="1.27" layer="26" font="vector" ratio="15" rot="MR0"/>
 <attribute name="VALUE" x="26.4" y="8.895" size="1.016" layer="28" rot="MR0"/>
 </element>
-<element name="C11" library="rcl" package="C0805K" value="15n" x="20.32" y="33.655" smashed="yes" rot="MR0">
+<element name="C11" library="rcl" package="C0805K" value="n.c." x="20.32" y="33.655" smashed="yes" rot="MR0">
 <attribute name="NAME" x="21.828" y="34.911" size="1.27" layer="26" font="vector" ratio="15" rot="MR0"/>
 <attribute name="VALUE" x="21.32" y="31.755" size="1.016" layer="28" rot="MR0"/>
 </element>
-<element name="C12" library="rcl" package="C0805K" value="15n" x="25.4" y="33.655" smashed="yes" rot="MR0">
+<element name="C12" library="rcl" package="C0805K" value="n.c." x="25.4" y="33.655" smashed="yes" rot="MR0">
 <attribute name="NAME" x="27.035" y="34.911" size="1.27" layer="26" font="vector" ratio="15" rot="MR0"/>
 <attribute name="VALUE" x="26.4" y="31.755" size="1.016" layer="28" rot="MR0"/>
 </element>
-<element name="AUDIO1" library="JACK3.5mm_FC6812x" package="FC68125" value="FC68125" x="4.699" y="52.705" smashed="yes"/>
+<element name="AUDIO1" library="JACK3.5mm_FC6812x" package="FC68125" value="FC68125" x="5.0038" y="52.705" smashed="yes"/>
 </elements>
 <signals>
@@
 <wire x1="1.836" y1="20.251" x2="1.836" y2="12.369" width="0.6096" layer="1"/>
 </signal>
-<signal name="POTX-2">
+<signal name="POTX-R">
 <contactref element="R3" pad="1"/>
 <contactref element="C5" pad="2"/>
@@
 <wire x1="39.37" y1="38.735" x2="39.37" y2="39.64" width="0.3048" layer="16"/>
 </signal>
-<signal name="POTY-2">
+<signal name="POTY-R">
 <contactref element="C6" pad="2"/>
 <contactref element="R4" pad="1"/>
@@
 <wire x1="35.56" y1="38.735" x2="35.56" y2="39.64" width="0.3048" layer="16"/>
 </signal>
-<signal name="POTX-1">
+<signal name="POTX-L">
 <contactref element="R1" pad="1"/>
 <contactref element="C3" pad="2"/>
@@
 <wire x1="39.37" y1="15.875" x2="39.37" y2="16.78" width="0.3048" layer="16"/>
 </signal>
-<signal name="POTY-1">
+<signal name="POTY-L">
 <contactref element="R2" pad="1"/>
 <contactref element="C4" pad="2"/>
@@
 <wire x1="11.175" y1="46.99" x2="9.525" y2="46.99" width="0.6096" layer="16"/>
 <via x="9.525" y="46.99" extent="1-16" drill="0.5"/>
-<wire x1="5.08" y1="46.99" x2="9.525" y2="46.99" width="0.6096" layer="1"/>
-<wire x1="1.849" y1="41.205" x2="1.849" y2="43.759" width="0.6096" layer="1"/>
-<wire x1="1.849" y1="43.759" x2="5.08" y2="46.99" width="0.6096" layer="1"/>
+<wire x1="9.525" y1="46.99" x2="5.08" y2="46.99" width="0.6096" layer="1"/>
+<wire x1="5.08" y1="46.99" x2="2.15" y2="44.06" width="0.6096" layer="1"/>
+<wire x1="2.15" y1="44.06" x2="2.1538" y2="41.205" width="0.6096" layer="1"/>
 </signal>
 <signal name="N$4">
@@
 <wire x1="8.89" y1="43.815" x2="10.795" y2="43.815" width="0.6096" layer="16"/>
 <wire x1="8.03" y1="49.305" x2="6.985" y2="48.26" width="0.6096" layer="16"/>
-<wire x1="8.03" y1="49.305" x2="8.099" y2="49.305" width="0.6096" layer="16"/>
+<wire x1="8.03" y1="49.305" x2="8.4038" y2="49.305" width="0.6096" layer="16"/>
 <wire x1="6.985" y1="48.26" x2="2.344" y2="48.26" width="0.6096" layer="16"/>
-<wire x1="2.344" y1="48.26" x2="1.299" y2="49.305" width="0.6096" layer="16"/>
+<wire x1="2.344" y1="48.26" x2="1.6038" y2="49.305" width="0.6096" layer="16"/>
 <wire x1="6.985" y1="48.26" x2="6.985" y2="45.72" width="0.6096" layer="16"/>
 <wire x1="6.985" y1="45.72" x2="8.89" y2="43.815" width="0.6096" layer="16"/>
@@
 </signal>
 </signals>
+<mfgpreviewcolors>
+<mfgpreviewcolor name="soldermaskcolor" color="0xC8008000"/>
+<mfgpreviewcolor name="silkscreencolor" color="0xFFFEFEFE"/>
+<mfgpreviewcolor name="backgroundcolor" color="0xFF282828"/>
+<mfgpreviewcolor name="coppercolor" color="0xFFFFBF00"/>
+<mfgpreviewcolor name="substratecolor" color="0xFF786E46"/>
+</mfgpreviewcolors>
 </board>
 </drawing>
